File: Schema/audio-and-video.kicad_sch (KiCad schematic)
At the start: 4 parts, among them U17 Kinect

Commit message: Robochallenge state
Other:
- title: (none) -> Audio and Video
Changed lines of the file:
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@@
 	(generator_version "8.0")
 	(paper "A4")
+	(title_block
+		(title "Audio and Video")
+		(date "08.05.2024")
+		(rev "1")
+		(comment 1 "The camera and audio schema")
+		(comment 2 "Takes handles audio input, audio output and video output")
+	)
 	(junction
 		(at 66.04 33.02)
